Commit message: new navigation

File: urdf/marrtinox.urdf (robot description, URDF)
Before this commit: robot marrtinox, 3 links, 2 joints
Links:
- link base_link: geometry collision box size=0.30 0.30 0.07; collision sphere radius=0.03
- link left_wheel: geometry collision cylinder length=0.02 radius=0.08; visual cylinder length=0.02 radius=0.08
- link right_wheel: geometry collision cylinder length=0.02 radius=0.08; visual cylinder length=0.02 radius=0.08
Joints:
- joint joint_left_wheel: origin xyz=0 0.30 0 rpy=0 0 0 -> xyz=0 0.16 0 rpy=0 0 0
- joint joint_right_wheel: origin xyz=0 -0.30 0 rpy=0 0 0 -> xyz=0 -0.16 0 rpy=0 0 0
